File: DIY Meshtastic 1W Node/DIY Meshtastic 1W Node.kicad_pcb (KiCad board)
At the start: 2 copper layers, 48.3 x 162.6 mm, 28 parts, among them J1 GPS CONNECTOR, J2 SSD1306 CONNECTOR, J3 I2C CONNECTOR 1, J4 I2C CONNECTOR 2, J5 I2C CONNECTOR 3, J6 I2C CONNECTOR 4, J7 Conn_Coaxial, J8 Conn_Coaxial, J9 Screw_Terminal_01x02, SW1 SW_Push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

Commit message: Modified the Schematic, and PCB
Added some documentation on the schematic and PCB, regenerated gerbers
Other:
- board text added: "+"
- board text added: "-"
- board text added: "30Vdc Max"
- board text added: "Gnd"
- board text added: "Tx"
