File: DIY Meshtastic 1W Node/DIY Meshtastic 1W Node.kicad_sch (KiCad schematic)
At the start: 24 parts, among them J1 GPS CONNECTOR, J2 SSD1306 CONNECTOR, J3 I2C CONNECTOR 1, J4 I2C CONNECTOR 2, J5 I2C CONNECTOR 3, J6 I2C CONNECTOR 4, J7 Conn_Coaxial, J8 Conn_Coaxial, J9 Screw_Terminal_01x02, SW1 SW_Push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

Commit message: Minor Change to the schematic
Add values for a couple of capacitors I forgot.
Parts:
- C10, C7, C8, C9: value C_Small -> 100nf
Changed lines of the file:
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@@
       (effects (font (size 1.27 1.27)) (justify left))
     )
-    (property "Value" "C_Small" (at 62.23 166.3763 0)
+    (property "Value" "100nf" (at 62.23 166.3763 0)
       (effects (font (size 1.27 1.27)) (justify left) hide)
     )
@@
       (effects (font (size 1.27 1.27)) (justify left))
     )
-    (property "Value" "C_Small" (at 49.53 116.8463 0)
+    (property "Value" "100nf" (at 49.53 116.8463 0)
       (effects (font (size 1.27 1.27)) (justify left) hide)
     )
@@
       (effects (font (size 1.27 1.27)) (justify left))
     )
-    (property "Value" "C_Small" (at 38.1 120.65 0)
+    (property "Value" "100nf" (at 38.1 120.65 0)
       (effects (font (size 1.27 1.27)) (justify left) hide)
     )
@@
       (effects (font (size 1.27 1.27)) (justify left))
     )
-    (property "Value" "C_Small" (at 54.61 168.9163 0)
+    (property "Value" "100nf" (at 54.61 168.9163 0)
       (effects (font (size 1.27 1.27)) (justify left) hide)
     )

Commit message: Modified the Schematic, and PCB
Added some documentation on the schematic and PCB, regenerated gerbers
Other:
- note added: "Set Meshtastic Firmare to the following Redefine GPS_RX_PIN = 16 Redefine GPS_TX_PIN = 17"
Changed lines of the file:
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@@
     (stroke (width 0) (type default))
+  )
+  (text "Set Meshtastic Firmare to the following\nRedefine GPS_RX_PIN = 16\nRedefine GPS_TX_PIN = 17"
+    (at 242.57 149.86 0)
+    (effects (font (size 1.27 1.27)) (justify left bottom))
   )
   (global_label "MISO" (shape input) (at 120.65 80.01 180) (fields_autoplaced)
